Commit message: updating launch files

File: binbot_bringup/urdf/binbot_robot.xacro (robot description, xacro)
@@ -2,5 +2,4 @@
 <robot
     name="binbot" xmlns:xacro="http://www.ros.org/wiki/xacro">
-  <xacro:include filename="$(find binbot_description)/urdf/binbot.gazebo"/>
   <link name="base_link"></link>
  <joint name="joint_base" type="fixed">
@@ -396,5 +395,5 @@
   </joint>
   <!--kinect_link-->
-  <link name="kinect_link">
+  <link name="camera_link">
       <inertial>
         <origin xyz="0.0 0.0 0.0" rpy="0.0 0.0 0.0"/>
@@ -417,15 +416,15 @@
   </link>
   <joint name="kinect_joint" type="fixed">
-    <origin xyz="0.28 0.0 0.01" rpy="0.0 0.0 0.0"/>
+    <origin xyz="0.24 0.0 0.452" rpy="0.0 0.0 0.0"/>
     <parent link="chassis_link"/>
-    <child link="kinect_link"/>
+    <child link="camera_link"/>
     <axis xyz="0.0 1 0.0"/>
   </joint>
-  <joint name="camera_optical_joint" type="fixed">
+ <joint name="camera_optical_joint" type="fixed">
     <origin xyz="0 0 0" rpy="-1.5707 0 -1.5707"/>
-    <parent link="kinect_link"/>
-    <child link="camera_link_optical"/>
-  </joint>
-  <link name="camera_link_optical">
+    <parent link="camera_link"/>
+    <child link="camera_depth_frame"/>
+  </joint>
+   <link name="camera_depth_frame">
   </link>
 </robot>

File: binbot_description/urdf/binbot_robot.xacro (robot description, xacro)
@@ -261,5 +261,5 @@
   </joint>
   <link
-    name="right_wheel">
+    name="rwheel">
     <inertial>
       <origin
@@ -301,5 +301,5 @@
   </link>
   <joint
-    name="right_wheel_joint"
+    name="base_to_rwheel"
     type="continuous">
     <origin
@@ -309,10 +309,10 @@
       link="chassis_link" />
     <child
-      link="right_wheel" />
+      link="rwheel" />
     <axis
       xyz="0 0 1" />
   </joint>
   <link
-    name="left_wheel">
+    name="lwheel">
    <inertial>
       <origin
@@ -354,5 +354,5 @@
   </link>
   <joint
-    name="left_wheel_joint"
+    name="base_to_lwheel"
     type="continuous">
     <origin
@@ -362,5 +362,5 @@
       link="chassis_link" />
     <child
-      link="left_wheel" />
+      link="lwheel" />
     <axis
       xyz="0 0 -1" />
@@ -396,5 +396,5 @@
   </joint>
   <!--kinect_link-->
-  <link name="kinect_link">
+  <link name="camera_link">
       <inertial>
         <origin xyz="0.0 0.0 0.0" rpy="0.0 0.0 0.0"/>
@@ -417,15 +417,22 @@
   </link>
   <joint name="kinect_joint" type="fixed">
-    <origin xyz="0.28 0.0 0.01" rpy="0.0 0.0 0.0"/>
+    <origin xyz="0.24 0.0 0.452" rpy="0.0 0.0 0.0"/>
     <parent link="chassis_link"/>
-    <child link="kinect_link"/>
+    <child link="camera_link"/>
     <axis xyz="0.0 1 0.0"/>
   </joint>
   <joint name="camera_optical_joint" type="fixed">
+      <origin xyz="0 0 0" rpy="-1.5707 0 -1.5707"/>
+      <parent link="camera_link"/>
+      <child link="camera_depth_frame"/>
+  </joint>
+  <link name="camera_depth_frame">
+  </link>
+  <!--joint name="camera_optical_joint2" type="fixed">
     <origin xyz="0 0 0" rpy="-1.5707 0 -1.5707"/>
-    <parent link="kinect_link"/>
-    <child link="camera_link_optical"/>
-  </joint>
-  <link name="camera_link_optical">
-  </link>
+    <parent link="camera_depth_frame"/>
+    <child link="camera_depth_optical_frame"/>
+  </joint>
+  <link name="camera_depth_optical_frame">
+  </link-->
 </robot>
